File: DigitalLogicWithSunPedal/DigitalLogicWithSunPedal.kicad_pcb (KiCad board)
At the start: 2 copper layers, 5 parts, among them IC1 REG1117-5, U2 TS881ICT, U3 TS881ICT, U4 TS881ICT, U5 TS881ICT

Commit message: Add files via upload
Parts:
- moved IC1 31.4 mm to (175.0, 91.0)
- moved U2 19.6 mm to (165.0, 97.0)
- moved U4 13.2 mm to (157.6, 88.0)
- moved U3 13.1 mm to (166.0, 88.0)
- moved U5 8.88 mm to (151.6, 88.0)
Routing:
- net +5V: track 7.92 -> 50.6 mm
- net +12V: track 0.00 -> 31.8 mm
- net GND: track 7.50 -> 34.6 mm
- net Net-(U4-+): track 0.00 -> 4.10 mm
- net Net-(U2--): track 5.60 -> 9.37 mm
Other:
- board outline added: 32 x 15 mm

Commit message: Add files via upload
Parts:
- added C1: CL21A106KOQNNNE, CL21A106KOQNNNE:CAPC2012X140N, F.Cu at (155.3, 113.0)
- added C2: CL21A106KOQNNNE, CL21A106KOQNNNE:CAPC2012X140N, F.Cu at (155.3, 116.0)
- added IC2: HEF4081BT,653, Package_SO:SOIC-14_3.9x8.7mm_P1.27mm, F.Cu at (148.8, 103.6)
- added J1: 776280-1, 776280-1:TE_776280-1, F.Cu at (114.7, 89.3)
- added J2: 4pin brake, DT15-4P:TE_DT15-4P, F.Cu at (113.6, 61.2)
- added J3: 4pin throttle, DT15-4P:TE_DT15-4P, F.Cu at (152.1, 61.2)
- added K1: J107F1AS123VDC.36, J107F1AS123VDC.36:RELAY_J107F1AS123VDC.36, F.Cu at (146.2, 89.8)
- added Q1: 2N2222A, 2N2222A:TO92254P470H750-3, F.Cu at (158.0, 107.2)
- added R10: CRCW08051K00FKEA, CRCW08051K00FKEA:RESC2012X50N, F.Cu at (138.1, 108.7)
- added R11: CRCW08051K00FKEA, CRCW08051K00FKEA:RESC2012X50N, F.Cu at (138.1, 111.7)
- added R12: CRCW08051K00FKEA, CRCW08051K00FKEA:RESC2012X50N, F.Cu at (138.1, 114.7)
- added R7: CRCW08051K00FKEA, CRCW08051K00FKEA:RESC2012X50N, F.Cu at (138.1, 99.8)
- added R8: CRCW08051K00FKEA, CRCW08051K00FKEA:RESC2012X50N, F.Cu at (138.1, 102.8)
- added R9: CRCW08051K00FKEA, CRCW08051K00FKEA:RESC2012X50N, F.Cu at (138.1, 105.8)
- moved U3 28.6 mm to (142.5, 104.3)
- moved U5 25.8 mm to (142.5, 112.1)
- moved U4 25.2 mm to (142.5, 108.2)
- moved U2 22.8 mm to (142.5, 100.3)
- moved IC1 20.1 mm to (158.4, 102.4)
Connections:
- U5 pad 3: +12V -> Net-(U4-+)
- U5 pad 4: Net-(U4-+) -> +12V
Routing:
- net +5V: track 50.6 -> 0.00 mm
- net GND: track 34.6 -> 0.00 mm
- net +12V: track 31.8 -> 0.00 mm
- net Net-(U2--): track 9.37 -> 0.00 mm
- net Net-(U4-+): track 4.10 -> 0.00 mm
Other:
- board outline removed

Commit message: Add files via upload
Parts:
- moved C2 78.5 mm to (199.8, 51.4), turned to 90 degrees
- moved J3 77.5 mm to (74.8, 55.9), turned to -90 degrees
- moved IC1 72.1 mm to (214.8, 57.5), turned to 90 degrees
- moved J1 68.8 mm to (183.5, 90.5), turned to 90 degrees
- moved R11 67.7 mm to (104.5, 53.0)
- moved C1 64.1 mm to (199.8, 67.0), turned to 90 degrees
- moved J2 63.8 mm to (73.7, 111.1)
- moved R10 56.2 mm to (89.5, 80.5), turned to 90 degrees
- moved U3 51.8 mm to (106.0, 67.5), turned to 90 degrees
- moved Q1 49.9 mm to (181.2, 63.0), turned to 90 degrees
- moved R12 45.9 mm to (135.6, 68.8), turned to 90 degrees
- moved U2 45.7 mm to (128.5, 56.9)
- moved K1 37.1 mm to (153.8, 53.5), turned to 180 degrees
- moved U4 32.9 mm to (111.2, 98.1), turned to -90 degrees
- moved U5 31.4 mm to (112.7, 122.1)
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Routing:
- net GND: track 0.00 -> 405.2 mm, vias 0 -> 4
- net +12V: track 0.00 -> 336.0 mm, vias 0 -> 4
- net +5V: track 0.00 -> 249.5 mm, vias 0 -> 4
- net Net-(U4-+): track 0.00 -> 154.2 mm, vias 0 -> 3
- net Net-(U2--): track 0.00 -> 126.7 mm
- net Net-(IC2-Pad2): track 0.00 -> 113.6 mm, vias 0 -> 2
- net Net-(IC2-Pad8): track 0.00 -> 80.4 mm
- net Net-(IC2-Pad3): track 0.00 -> 58.2 mm, vias 0 -> 2
- net Net-(J1-Pad8): track 0.00 -> 57.9 mm
- net Net-(IC2-Pad4): track 0.00 -> 57.0 mm, vias 0 -> 2
- net Net-(J1-Pad7): track 0.00 -> 56.4 mm
- net Net-(IC2-Pad1): track 0.00 -> 48.6 mm, vias 0 -> 4
- net Net-(IC2-Pad5): track 0.00 -> 37.0 mm
- net Net-(K1-PadCOIL1): track 0.00 -> 26.2 mm
- net Net-(IC2-Pad10): track 0.00 -> 24.9 mm
Other:
- board outline added: 173 x 100.5 mm

Commit message: Add files via upload
Parts:
- moved IC1 33.2 mm to (182.5, 50.0), turned to 0 degrees
- moved C1 32.5 mm to (170.0, 54.1), turned to -90 degrees
- moved C2 30.7 mm to (170.0, 44.1)
Routing:
- net GND: track 405.2 -> 487.6 mm, vias 4 -> 22
- net +5V: track 249.5 -> 219.5 mm
- net +12V: track 336.0 -> 341.2 mm
- added copper zone on B.Cu, net GND
Other:
- board size 173 x 100.5 mm -> 155 x 110 mm

Commit message: Add files via upload
Parts:
- removed J3: 4pin throttle, DT15-4P:TE_DT15-4P
- J2: value 4pin brake -> 776280-1; footprint DT15-4P:TE_DT15-4P -> 776280-1:TE_776280-1
- moved R10 67.0 mm to (156.5, 82.5), turned to 180 degrees
- moved J2 57.7 mm to (122.3, 80.0), turned to -90 degrees
- moved R11 55.3 mm to (154.2, 77.2), turned to 90 degrees
- moved C2 52.4 mm to (158.8, 95.2), turned to -90 degrees
- moved K1 50.8 mm to (141.5, 102.8)
- moved IC1 48.3 mm to (168.8, 96.2), turned to 180 degrees
- moved U5 47.5 mm to (147.8, 90.0)
- moved C1 45.9 mm to (161.8, 99.2)
- moved U3 43.9 mm to (148.8, 77.5), turned to 180 degrees
- moved Q1 43.3 mm to (169.5, 104.7), turned to 0 degrees
- moved U4 42.6 mm to (153.0, 90.0), turned to 0 degrees
- moved R7 28.9 mm to (153.2, 86.8), turned to 0 degrees
- moved U2 26.4 mm to (150.2, 71.8)
- moved IC2 25.3 mm to (166.2, 81.0)
- moved R8 19.5 mm to (142.0, 88.2), turned to -90 degrees
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Connections:
- J2 pad 2: Net-(U4-+) -> Net-(U2--)
Routing:
- net GND: track 487.6 -> 55.2 mm, vias 22 -> 8
- net +12V: track 341.2 -> 203.6 mm, vias 4 -> 0
- net +5V: track 219.5 -> 108.3 mm, vias 4 -> 3
- net Net-(IC2-Pad2): track 113.6 -> 14.2 mm, vias 2 -> 0
- net Net-(U2--): track 126.7 -> 61.2 mm
- net Net-(U4-+): track 154.2 -> 99.6 mm, vias 3 -> 2
- net Net-(IC2-Pad3): track 58.2 -> 17.3 mm, vias 2 -> 0
- net Net-(IC2-Pad8): track 80.1 -> 44.4 mm, vias 0 -> 1
- net Net-(IC2-Pad4): track 57.0 -> 26.1 mm, vias 2 -> 0
- net Net-(J1-Pad8): track 57.9 -> 88.2 mm
- net Net-(IC2-Pad1): track 48.6 -> 24.0 mm, vias 4 -> 2
- net Net-(IC2-Pad5): track 37.0 -> 17.6 mm
- net Net-(IC2-Pad10): track 24.9 -> 10.4 mm
- net Net-(J1-Pad7): track 56.4 -> 66.4 mm
- net Net-(K1-PadCOIL1): track 26.2 -> 20.2 mm
Other:
- board size 155 x 110 mm -> 82.5 x 67 mm
